File: 20 Pin Electrode Connector/20PinElectrodeConnector/20PinElectrodeConnector.sch (KiCad schematic (older format))
At the start: 21 parts, among them J1 Conn_02x10_Odd_Even

Commit message: Conform to microscope stage bracket.
Parts:
- TP1, TP10, TP11, TP12, TP13, TP14, TP15, TP16, TP17, TP18, TP19, TP2, TP20, TP3, TP4, TP5, TP6, TP7, TP8, TP9: footprint Connector_Wire:SolderWire-0.25sqmm_1x01_D0.65mm_OD2mm_Relief -> Connector_Wire:SolderWire-0.25sqmm_1x01_D0.65mm_OD2mm
