File: SMU Test Fixture/power_supplies.sch (KiCad schematic (older format))
At the start: 42 parts, among them J13 Hot_Spade, J14 Power Outputs, J15 Neutral_Spade, T1 VPP28-1060, U10 LT3045xMSE-1, U11 LT1086-12, U12 LT3094xMSE, U9 LT1086-5.0

Commit message: Update LT3045 symbol w/ missing pins.
Parts:
- U10: value LT3045xMSE-1 -> MAGI_Symbols_LT3045xMSE-1; symbol MAGI_Symbols:LT3045xMSE-1 -> MAGI_Symbols:LT3045xMSE
Connections:
- wire segments 201 -> 209
- no-connect marks 4 -> 5
Other:
- moved on the sheet: C35, C36, C40, R37, R38
Changed lines of the file:
@@
 L Device:R_Small_US R37
 U 1 1 5FC9A651
-P 1900 4350
-F 0 "R37" H 1968 4396 50  0000 L CNN
-F 1 "150k" H 1925 4275 50  0000 L CNN
-F 2 "Resistor_SMD:R_0805_2012Metric_Pad1.20x1.40mm_HandSolder" H 1900 4350 50  0001 C CNN
-F 3 "~" H 1900 4350 50  0001 C CNN
-	1    1900 4350
+P 1900 4375
+F 0 "R37" H 1968 4421 50  0000 L CNN
+F 1 "150k" H 1925 4300 50  0000 L CNN
+F 2 "Resistor_SMD:R_0805_2012Metric_Pad1.20x1.40mm_HandSolder" H 1900 4375 50  0001 C CNN
+F 3 "~" H 1900 4375 50  0001 C CNN
+	1    1900 4375
 	-1   0    0    -1
 $EndComp
@@
 L Device:R_Small_US R38
 U 1 1 5FC9B12D
-P 1925 5975
-F 0 "R38" H 1993 6021 50  0000 L CNN
-F 1 "150k" H 1950 5900 50  0000 L CNN
-F 2 "Resistor_SMD:R_0805_2012Metric_Pad1.20x1.40mm_HandSolder" H 1925 5975 50  0001 C CNN
-F 3 "~" H 1925 5975 50  0001 C CNN
-	1    1925 5975
+P 1775 5975
+F 0 "R38" H 1843 6021 50  0000 L CNN
+F 1 "150k" H 1800 5900 50  0000 L CNN
+F 2 "Resistor_SMD:R_0805_2012Metric_Pad1.20x1.40mm_HandSolder" H 1775 5975 50  0001 C CNN
+F 3 "~" H 1775 5975 50  0001 C CNN
+	1    1775 5975
 	-1   0    0    -1
 $EndComp
 Wire Wire Line
-	1900 4250 1900 4200
-Wire Wire Line
-	1900 4450 1900 4500
-Wire Wire Line
-	1925 6075 1925 6125
+	1900 4275 1900 4225
+Wire Wire Line
+	1900 4475 1900 4500
+Wire Wire Line
+	1775 6075 1775 6125
 $Comp
 L Device:C_Small C35
 U 1 1 5FCA03E8
-P 2150 4350
-F 0 "C35" H 2000 4450 50  0000 L CNN
-F 1 "22u" H 2000 4275 50  0000 L CNN
-F 2 "Capacitor_SMD:C_0805_2012Metric_Pad1.18x1.45mm_HandSolder" H 2150 4350 50  0001 C CNN
-F 3 "~" H 2150 4350 50  0001 C CNN
-	1    2150 4350
+P 2150 4375
+F 0 "C35" H 2000 4475 50  0000 L CNN
+F 1 "22u" H 2000 4300 50  0000 L CNN
+F 2 "Capacitor_SMD:C_0805_2012Metric_Pad1.18x1.45mm_HandSolder" H 2150 4375 50  0001 C CNN
+F 3 "~" H 2150 4375 50  0001 C CNN
+	1    2150 4375
 	1    0    0    -1
 $EndComp
@@
 L Device:C_Small C36
 U 1 1 5FCA1017
-P 2175 5975
-F 0 "C36" H 2025 6050 50  0000 L CNN
-F 1 "22u" H 2025 5900 50  0000 L CNN
-F 2 "Capacitor_SMD:C_0805_2012Metric_Pad1.18x1.45mm_HandSolder" H 2175 5975 50  0001 C CNN
-F 3 "~" H 2175 5975 50  0001 C CNN
-	1    2175 5975
-	1    0    0    -1
-$EndComp
-Wire Wire Line
-	2175 5875 2175 5825
-Wire Wire Line
-	2175 5825 2050 5825
-Wire Wire Line
-	1925 5825 1925 5875
-Wire Wire Line
-	2175 6075 2175 6125
-Wire Wire Line
-	2175 6125 1925 6125
-Connection ~ 1925 6125
-Wire Wire Line
-	2150 4450 2150 4500
+P 2025 5975
+F 0 "C36" H 1875 6050 50  0000 L CNN
+F 1 "22u" H 1875 5900 50  0000 L CNN
+F 2 "Capacitor_SMD:C_0805_2012Metric_Pad1.18x1.45mm_HandSolder" H 2025 5975 50  0001 C CNN
+F 3 "~" H 2025 5975 50  0001 C CNN
+	1    2025 5975
+	1    0    0    -1
+$EndComp
+Wire Wire Line
+	2025 5875 2025 5825
+Wire Wire Line
+	1775 5825 1775 5875
+Wire Wire Line
+	2025 6075 2025 6125
+Wire Wire Line
+	2025 6125 1900 6125
+Wire Wire Line
+	2150 4475 2150 4500
 Wire Wire Line
 	2150 4500 2025 4500
 Wire Wire Line
-	2150 4250 2150 4200
-Wire Wire Line
-	2150 4200 1900 4200
-Connection ~ 1900 4200
+	2150 4275 2150 4225
+Wire Wire Line
+	2150 4225 1900 4225
+Connection ~ 1900 4225
 Connection ~ 1800 3700
 Wire Wire Line
 	1800 3700 1800 3750
 Wire Wire Line
-	2875 6875 1850 6875
-Wire Wire Line
-	1850 6625 1850 6675
-Connection ~ 1850 6675
+	2875 6875 1750 6875
 Wire Wire Line
 	2800 6625 2800 6725
@@
 $EndComp
 Wire Wire Line
-	1600 6675 1600 6300
+	1550 6675 1550 6300
 $Comp
 L Device:CP_Small C29
@@
 $EndComp
 Wire Wire Line
-	1600 5675 1600 6100
+	1550 5675 1550 6100
 $Comp
 L Device:C_Small C40
 U 1 1 60124B22
-P 1600 6200
-F 0 "C40" H 1692 6246 50  0000 L CNN
-F 1 "4.7u" H 1692 6155 50  0000 L CNN
-F 2 "Capacitor_SMD:C_0805_2012Metric_Pad1.18x1.45mm_HandSolder" H 1600 6200 50  0001 C CNN
-F 3 "~" H 1600 6200 50  0001 C CNN
-	1    1600 6200
+P 1550 6200
+F 0 "C40" H 1642 6246 50  0000 L CNN
+F 1 "4.7u" H 1642 6155 50  0000 L CNN
+F 2 "Capacitor_SMD:C_0805_2012Metric_Pad1.18x1.45mm_HandSolder" H 1550 6200 50  0001 C CNN
+F 3 "~" H 1550 6200 50  0001 C CNN
+	1    1550 6200
 	-1   0    0    -1
 $EndComp
-Wire Wire Line
-	2850 3550 2850 3850
 Wire Wire Line
 	2875 6525 2875 6875
@@
 	1550 3700 1625 3700
 Wire Wire Line
-	1575 6675 1600 6675
-Connection ~ 1600 6675
-Wire Wire Line
-	1600 6675 1850 6675
+	1500 6675 1550 6675
 Wire Wire Line
 	1625 4650 1625 4325
@@
 	4825 1550 4825 1525
 Wire Wire Line
-	1925 6125 1925 6325
+	2725 6525 2875 6525
 NoConn ~ 1925 6425
 Wire Wire Line
-	2875 6425 2725 6425
-Wire Wire Line
-	2725 6525 2875 6525
-NoConn ~ 1925 6525
-Wire Wire Line
-	1925 6625 1850 6625
-Wire Wire Line
 	2725 6625 2800 6625
 Wire Wire Line
 	2800 6725 2725 6725
 Wire Wire Line
-	1900 4200 1900 4050
-Wire Wire Line
-	2700 3850 2850 3850
+	1900 4225 1900 4150
 Wire Wire Line
 	2850 3950 2700 3950
@@
 $EndComp
 $Comp
-L MAGI_Symbols:LT3045xMSE-1 U10
+L MAGI_Symbols:LT3045xMSE U10
 U 1 1 5FC8B975
 P 2300 3800
@@
 AR Path="/64A89145/5FC8B975" Ref="U10"  Part="1"
 F 0 "U10" H 2300 4281 50  0000 C CNN
-F 1 "LT3045xMSE-1" H 2300 4190 50  0000 C CNN
+F 1 "MAGI_Symbols_LT3045xMSE-1" H 2300 4190 50  0000 C CNN
 F 2 "Package_SO:MSOP-12-1EP_3x4mm_P0.65mm_EP1.65x2.85mm" H 2300 4125 50  0001 C CNN
 F 3 "https://www.analog.com/media/en/technical-documentation/data-sheets/3045fa.pdf" H 2300 3800 50  0001 C CNN
@@
 Wire Wire Line
 	2025 4500 1900 4500
-Wire Wire Line
-	2850 3950 2850 4650
 Wire Wire Line
 	3075 4300 3075 4650
@@
 unreg_pos_18VDC
 Wire Wire Line
-	2050 5825 2050 5675
-Connection ~ 2050 5825
-Wire Wire Line
-	2050 5825 1925 5825
-Wire Wire Line
 	2325 6125 2325 5675
 Wire Wire Line
-	2875 6425 2875 5675
-Wire Wire Line
 	3100 6000 3100 5675
-Wire Wire Line
-	3100 5675 2875 5675
-Wire Wire Line
-	2875 5675 2575 5675
-Connection ~ 2875 5675
-Wire Wire Line
-	2325 5675 2050 5675
-Connection ~ 2325 5675
-Wire Wire Line
-	2050 5675 1600 5675
-Connection ~ 2050 5675
-Text Label 1575 6675 2    50   ~ 10
+Text Label 1500 6675 2    50   ~ 10
 unreg_neg_18VDC
 $Comp
@@
 	2650 5425 2650 5450
 Connection ~ 2575 5675
-Wire Wire Line
-	2575 5675 2325 5675
 $Comp
 L power:+15V #PWR074
@@
 To BZH01/Z0000/01\nSwitchable, fused, power entry module\n3.5A Slow Blow
 Wire Wire Line
-	2025 4650 2300 4650
-Wire Wire Line
-	2300 4200 2300 4650
-Connection ~ 2300 4650
+	2250 4300 2250 4375
 Wire Wire Line
 	5725 3600 5475 3600
@@
 	6025 3900 6025 3950
 Connection ~ 6025 3950
-Wire Wire Line
-	1850 6675 1850 6725
-Wire Wire Line
-	1925 6725 1850 6725
-Connection ~ 1850 6725
-Wire Wire Line
-	1850 6725 1850 6875
-Wire Wire Line
-	2300 4650 2550 4650
 Wire Wire Line
 	2550 4650 2550 4725
@@
 	1    0    0    -1
 $EndComp
+Wire Wire Line
+	1775 5825 1900 5825
+Wire Wire Line
+	1750 6675 1750 6700
+Wire Wire Line
+	1900 5825 1900 5675
+Connection ~ 1900 5825
+Wire Wire Line
+	1900 5825 2025 5825
+Wire Wire Line
+	1900 6325 1900 6125
+Connection ~ 1900 6125
+Wire Wire Line
+	1900 6125 1775 6125
+Wire Wire Line
+	1900 6625 1925 6625
+Wire Wire Line
+	1900 6625 1900 6700
+Wire Wire Line
+	1900 6725 1925 6725
+Wire Wire Line
+	1750 6700 1900 6700
+Connection ~ 1750 6700
+Wire Wire Line
+	1750 6700 1750 6875
+Connection ~ 1900 6700
+Wire Wire Line
+	1900 6700 1900 6725
+Connection ~ 1550 6675
+Wire Wire Line
+	1550 6675 1750 6675
+Connection ~ 2325 5675
+Wire Wire Line
+	2325 5675 2575 5675
+Wire Wire Line
+	2575 5675 2725 5675
+Wire Wire Line
+	1550 5675 1900 5675
+Wire Wire Line
+	1900 6325 1925 6325
+Connection ~ 1900 5675
+Wire Wire Line
+	1900 5675 2325 5675
+NoConn ~ 1925 6525
+Wire Wire Line
+	2725 6425 2725 5675
+Connection ~ 2725 5675
+Wire Wire Line
+	2725 5675 3100 5675
+Wire Wire Line
+	2025 4650 2250 4650
+Connection ~ 2250 4650
+Wire Wire Line
+	2250 4650 2550 4650
+Wire Wire Line
+	2250 4375 2350 4375
+Wire Wire Line
+	2350 4375 2350 4300
+Connection ~ 2250 4375
+Wire Wire Line
+	2250 4375 2250 4650
+NoConn ~ 1900 4050
+Wire Wire Line
+	2700 4050 2850 4050
+Wire Wire Line
+	2850 4050 2850 4650
+Wire Wire Line
+	2850 3550 2850 3950
+Wire Wire Line
+	2700 3850 2775 3850
+Wire Wire Line
+	2775 3850 2775 3750
+Connection ~ 2775 3750
 $EndSCHEMATC

Commit message: Back to kelvin connection on +-15 reg out cap
Parts:
- C33, C39: footprint Capacitor_SMD:C_0805_2012Metric_Pad1.18x1.45mm_HandSolder -> MAGI_Footprints:C_0805_2012Metric_Pad1.18x1.45mm_HandSolder_Kelvin
- U10: value MAGI_Symbols_LT3045xMSE-1 -> LT3045
- U12: value LT3094xMSE -> LT3094
Changed lines of the file:
@@
 F 0 "C33" H 3167 4246 50  0000 L CNN
 F 1 "10u" H 3167 4155 50  0000 L CNN
-F 2 "Capacitor_SMD:C_0805_2012Metric_Pad1.18x1.45mm_HandSolder" H 3075 4200 50  0001 C CNN
+F 2 "MAGI_Footprints:C_0805_2012Metric_Pad1.18x1.45mm_HandSolder_Kelvin" H 3075 4200 50  0001 C CNN
 F 3 "~" H 3075 4200 50  0001 C CNN
 	1    3075 4200
@@
 F 0 "C39" H 3192 6146 50  0000 L CNN
 F 1 "10u" H 3192 6055 50  0000 L CNN
-F 2 "Capacitor_SMD:C_0805_2012Metric_Pad1.18x1.45mm_HandSolder" H 3100 6100 50  0001 C CNN
+F 2 "MAGI_Footprints:C_0805_2012Metric_Pad1.18x1.45mm_HandSolder_Kelvin" H 3100 6100 50  0001 C CNN
 F 3 "~" H 3100 6100 50  0001 C CNN
 	1    3100 6100
@@
 P 2325 6525
 F 0 "U12" H 2325 7025 50  0000 C CNN
-F 1 "LT3094xMSE" H 2325 7125 50  0000 C CNN
+F 1 "LT3094" H 2325 7125 50  0000 C CNN
 F 2 "Package_SO:MSOP-12-1EP_3x4mm_P0.65mm_EP1.65x2.85mm" H 2325 6950 50  0001 C CNN
 F 3 "https://www.analog.com/media/en/technical-documentation/data-sheets/LT3094.pdf" H 2325 6625 50  0001 C CNN
@@
 AR Path="/64A89145/5FC8B975" Ref="U10"  Part="1"
 F 0 "U10" H 2300 4281 50  0000 C CNN
-F 1 "MAGI_Symbols_LT3045xMSE-1" H 2300 4190 50  0000 C CNN
+F 1 "LT3045" H 2300 4190 50  0000 C CNN
 F 2 "Package_SO:MSOP-12-1EP_3x4mm_P0.65mm_EP1.65x2.85mm" H 2300 4125 50  0001 C CNN
 F 3 "https://www.analog.com/media/en/technical-documentation/data-sheets/3045fa.pdf" H 2300 3800 50  0001 C CNN

Commit message: Add crowbar protection for regulator inputs.
Parts:
- removed D39: 20V Clamp, Package_TO_SOT_SMD:SOT-323_SC-70_Handsoldering, symbol Device:D_TVS_x2_AAC
- added D39, D46: 20V, Diode_SMD:D_SOD-523, symbol Device:D_Zener
- added Q1, Q2: IRFL014, Package_TO_SOT_SMD:SOT-223, symbol Device:Q_NMOS_GDSD
- added R39, R40: 1K, Resistor_SMD:R_0805_2012Metric_Pad1.20x1.40mm_HandSolder, symbol Device:R_Small_US
Connections:
- net labels added: unfilt_neg, unfilt_pos
- wire segments 209 -> 230
Other:
- note added: "LT3045 bottom pad is input.\nUse thermal jumpers to\nconduct heat into ground."
- note added: "Mains Input and Rectification"
- note added: "OVP"
- note removed: "LT3045 bottom pad is input.\nUse thermal jumpers to\nconduct into ground."
- note removed: "Mains input and rectification"
- moved on the sheet: R33, R34, R35, R36, U11

Commit message: Daisy-chain 12V->5V regs.
Changed lines of the file:
@@
 	3475 6825 3475 6725
-Wire Wire Line
-	5400 3600 5475 3600
-Text Label 5400 3600 2    50   ~ 10
-unreg_pos_18VDC
 Wire Wire Line
 	5400 5725 5475 5725
@@
 Wire Wire Line
 	5725 3600 5475 3600
-Connection ~ 5475 3600
 Wire Wire Line
 	6025 3900 6025 3950
@@
 Text Notes 9100 725  0    118  ~ 24
 OVP
+$Comp
+L power:+12V #PWR?
+U 1 1 60F40CB4
+P 5475 3550
+F 0 "#PWR?" H 5475 3400 50  0001 C CNN
+F 1 "+12V" H 5490 3723 50  0000 C CNN
+F 2 "" H 5475 3550 50  0001 C CNN
+F 3 "" H 5475 3550 50  0001 C CNN
+	1    5475 3550
+	1    0    0    -1
+$EndComp
+Wire Wire Line
+	5475 3600 5475 3550
+Connection ~ 5475 3600
 $EndSCHEMATC

Commit message: Improved crowbar performance. Posted for reddit design review.
Parts:
- D39, D46: value 20V -> 16V; PN BZX584C20-G3-08 -> BZX584C16-G3-08
- F1: footprint Fuse:Fuse_1812_4532Metric -> Fuse:Fuse_2920_7451Metric_Pad2.10x5.45mm_HandSolder; PN 1812L050/30PR -> 2920L110/60MR
- F2: value 1 A -> 500mA; PN 1812L050/30PR -> 1812L050/60
- R39, R40: value 1K -> 180R
- TH1: value 3.5A max <130C -> 2.5A max, 33R @ 25C; footprint MAGI_Footprints:NTC d=11.5 p=5mm w=6mm -> MAGI_Footprints:NTC d=15 p=7p5mm w=7mm; PN B57236S0100M000 -> B57237S0330M051
Other:
- note added: "+ 12 V for Relays"
- note added: "+ 15V for Analog Section"
- note added: "+ 5V for Aux / pH Meter"
- note added: "- 15V for Analog Section"
- note added: "Overvoltage Protection"
- note added: "Spice model results for:\nBZX584C16-G3-08\nIFRL014\n180R\n=> 1A polyfuse trips in 4s @ Is=3A @ 22V unreg output.\n=> +10% expected unreg voltage => Is = 180mA\n\nPrevent overvoltage damage to\n LT3045, 3094 absmax Vin=22V."
- note added: "To BZH01/Z0000/01\nSwitchable, fused, power entry module\n2.5A Slow Blow"
- note removed: "+ 12 V for relays"
- note removed: "+ 15V for analog section"
- note removed: "+ 5V for aux / pH meter"
- note removed: "- 15V for analog section"
- note removed: "OVP"
- note removed: "To BZH01/Z0000/01\nSwitchable, fused, power entry module\n3.5A Slow Blow"
- moved on the sheet: C33, C34, C35, C36, C39, C40, R37, R38, U11, U12, U9

Commit message: Replace crowbar with LTC2966.
Parts:
- removed D39, D46: 16V, Diode_SMD:D_SOD-523, symbol Device:D_Zener
- removed Q1, Q2: IRFL014, Package_TO_SOT_SMD:SOT-223, symbol Device:Q_NMOS_GDSD
- removed R39, R40: 180R, Resistor_SMD:R_0805_2012Metric_Pad1.20x1.40mm_HandSolder, symbol Device:R_Small_US
- added Q? (x2): NTD5865NL, Package_TO_SOT_SMD:TO-252-3_TabPin4, symbol Device:Q_NMOS_GDSD
- added R?: 4.02k, symbol Device:R_Small_US
- added R?: 845R, symbol Device:R_Small_US
- added R? (x2): 46.4K, symbol Device:R_Small_US
- added R?: 4.96K, symbol Device:R_Small_US
- added R?: 4.64K, symbol Device:R_Small_US
- added R? (x2): 100R, symbol Device:R_Small_US
- added R? (x2): 100K, symbol Device:R_Small_US
- added U?: LTC2966CSWPBF, MAGI_Footprints:SO-20_SW, symbol MAGI_Symbols:LTC2966CSWPBF
Connections:
- net labels added: neg_disable, ovp_ref, pos_disable
- net labels removed: unfilt_neg, unfilt_pos
- wire segments 230 -> 256
Other:
- note added: "High threshold: ±22 V\nLow threshold: ±20 V"
- note removed: "Spice model results for:\nBZX584C16-G3-08\nIFRL014\n180R\n=> 1A polyfuse trips in 4s @ Is=3A @ 22V unreg output.\n=> +10% expected unreg voltage => Is = 180mA\n\nPrevent overvoltage damage to\n LT3045, 3094 absmax Vin=22V."
- moved on the sheet: C27, C28, C29, C30, C33, C34, C35, C36, C39, C40, D37, D38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

Commit message: Increase ptc fuse size to 3.7 A, update FPs.
Parts:
- F1: value 1 A -> 3.7 A; PN 2920L110/60MR -> 2920L185
- F2: value 500mA -> 3.7 A; footprint Fuse:Fuse_1812_4532Metric -> Fuse:Fuse_2920_7451Metric_Pad2.10x5.45mm_HandSolder; PN 1812L050/60 -> 2920L185
- R39, R40, R41, R42, R43, R44, R45, R46, R47, R48: renamed from R?; footprint (none) -> Resistor_SMD:R_0805_2012Metric_Pad1.20x1.40mm_HandSolder
- gave numbers to parts that had none: 3
Changed lines of the file:
@@
 P 3900 1700
 F 0 "F2" V 4000 1700 50  0000 C CNN
-F 1 "500mA" V 4075 1700 50  0000 C CNN
-F 2 "Fuse:Fuse_1812_4532Metric" H 3950 1500 50  0001 L CNN
-F 3 "https://www.mouser.com/datasheet/2/240/Littelfuse_PTC_1812L_Datasheet.pdf-693388.pdf" H 3900 1700 50  0001 C CNN
-F 4 "1812L050/60" V 3900 1700 50  0001 C CNN "PN"
+F 1 "3.7 A" V 4075 1700 50  0000 C CNN
+F 2 "Fuse:Fuse_2920_7451Metric_Pad2.10x5.45mm_HandSolder" H 3950 1500 50  0001 L CNN
+F 3 "https://www.mouser.com/datasheet/2/240/Littelfuse_PTC_2920L_Datasheet.pdf-365479.pdf" H 3900 1700 50  0001 C CNN
+F 4 "2920L185" V 3900 1700 50  0001 C CNN "PN"
 	1    3900 1700
 	0    1    1    0
@@
 P 3900 1500
 F 0 "F1" V 3675 1500 50  0000 C CNN
-F 1 "1 A" V 3766 1500 50  0000 C CNN
+F 1 "3.7 A" V 3766 1500 50  0000 C CNN
 F 2 "Fuse:Fuse_2920_7451Metric_Pad2.10x5.45mm_HandSolder" H 3950 1300 50  0001 L CNN
 F 3 "https://www.mouser.com/datasheet/2/240/Littelfuse_PTC_2920L_Datasheet.pdf-365479.pdf" H 3900 1500 50  0001 C CNN
-F 4 " 2920L110/60MR " V 3900 1500 50  0001 C CNN "PN"
+F 4 "2920L185" V 3900 1500 50  0001 C CNN "PN"
 	1    3900 1500
 	0    1    1    0
@@
 Connection ~ 9350 3100
 $Comp
-L power:GND #PWR?
+L power:GND #PWR085
 U 1 1 6072D966
 P 9725 3125
-F 0 "#PWR?" H 9725 2875 50  0001 C CNN
+F 0 "#PWR085" H 9725 2875 50  0001 C CNN
 F 1 "GND" H 9730 2952 50  0000 C CNN
 F 2 "" H 9725 3125 50  0001 C CNN
@@
 ovp_ref
 $Comp
-L Device:R_Small_US R?
+L Device:R_Small_US R45
 U 1 1 607B7E7A
 P 7300 2200
-F 0 "R?" H 7368 2246 50  0000 L CNN
+F 0 "R45" H 7368 2246 50  0000 L CNN
 F 1 "4.02k" H 7368 2155 50  0000 L CNN
-F 2 "" H 7300 2200 50  0001 C CNN
+F 2 "Resistor_SMD:R_0805_2012Metric_Pad1.20x1.40mm_HandSolder" H 7300 2200 50  0001 C CNN
 F 3 "~" H 7300 2200 50  0001 C CNN
 	1    7300 2200
@@
 $EndComp
 $Comp
-L Device:R_Small_US R?
+L Device:R_Small_US R47
 U 1 1 607B853F
 P 7300 2450
-F 0 "R?" H 7368 2496 50  0000 L CNN
+F 0 "R47" H 7368 2496 50  0000 L CNN
 F 1 "845R" H 7368 2405 50  0000 L CNN
-F 2 "" H 7300 2450 50  0001 C CNN
+F 2 "Resistor_SMD:R_0805_2012Metric_Pad1.20x1.40mm_HandSolder" H 7300 2450 50  0001 C CNN
 F 3 "~" H 7300 2450 50  0001 C CNN
 	1    7300 2450
@@
 $EndComp
 $Comp
-L Device:R_Small_US R?
+L Device:R_Small_US R48
 U 1 1 607BAE77
 P 7300 2700
-F 0 "R?" H 7368 2746 50  0000 L CNN
+F 0 "R48" H 7368 2746 50  0000 L CNN
 F 1 "46.4K" H 7368 2655 50  0000 L CNN
-F 2 "" H 7300 2700 50  0001 C CNN
+F 2 "Resistor_SMD:R_0805_2012Metric_Pad1.20x1.40mm_HandSolder" H 7300 2700 50  0001 C CNN
 F 3 "~" H 7300 2700 50  0001 C CNN
 	1    7300 2700
@@
 $EndComp
 $Comp
-L Device:R_Small_US R?
+L Device:R_Small_US R40
 U 1 1 607BB513
 P 6850 1750
-F 0 "R?" H 6918 1796 50  0000 L CNN
+F 0 "R40" H 6918 1796 50  0000 L CNN
 F 1 "4.96K" H 6918 1705 50  0000 L CNN
-F 2 "" H 6850 1750 50  0001 C CNN
+F 2 "Resistor_SMD:R_0805_2012Metric_Pad1.20x1.40mm_HandSolder" H 6850 1750 50  0001 C CNN
 F 3 "~" H 6850 1750 50  0001 C CNN
 	1    6850 1750
@@
 $EndComp
 $Comp
-L Device:R_Small_US R?
+L Device:R_Small_US R42
 U 1 1 607BBB9F
 P 6850 2000
-F 0 "R?" H 6918 2046 50  0000 L CNN
+F 0 "R42" H 6918 2046 50  0000 L CNN
 F 1 "46.4K" H 6918 1955 50  0000 L CNN
-F 2 "" H 6850 2000 50  0001 C CNN
+F 2 "Resistor_SMD:R_0805_2012Metric_Pad1.20x1.40mm_HandSolder" H 6850 2000 50  0001 C CNN
 F 3 "~" H 6850 2000 50  0001 C CNN
 	1    6850 2000
@@
 $EndComp
 $Comp
-L Device:R_Small_US R?
+L Device:R_Small_US R46
 U 1 1 607BBF21
 P 6850 2250
-F 0 "R?" H 6918 2296 50  0000 L CNN
+F 0 "R46" H 6918 2296 50  0000 L CNN
 F 1 "4.64K" H 6918 2205 50  0000 L CNN
-F 2 "" H 6850 2250 50  0001 C CNN
+F 2 "Resistor_SMD:R_0805_2012Metric_Pad1.20x1.40mm_HandSolder" H 6850 2250 50  0001 C CNN
 F 3 "~" H 6850 2250 50  0001 C CNN
 	1    6850 2250
@@
 	7550 1650 7550 1525
 $Comp
-L power:GND #PWR?
+L power:GND #PWR084
 U 1 1 60837A92
 P 6850 2600
-F 0 "#PWR?" H 6850 2350 50  0001 C CNN
+F 0 "#PWR084" H 6850 2350 50  0001 C CNN
 F 1 "GND" H 6855 2427 50  0000 C CNN
 F 2 "" H 6850 2600 50  0001 C CNN
@@
 	8400 1150 8400 1100
 $Comp
-L Device:Q_NMOS_GDSD Q?
+L Device:Q_NMOS_GDSD Q1
 U 1 1 60963764
 P 4425 1350
-F 0 "Q?" V 4325 1450 50  0000 C CNN
+F 0 "Q1" V 4325 1450 50  0000 C CNN
 F 1 "NTD5865NL" V 4250 1575 50  0000 C CNN
 F 2 "Package_TO_SOT_SMD:TO-252-3_TabPin4" H 4625 1450 50  0001 C CNN
@@
 $EndComp
 $Comp
-L Device:Q_NMOS_GDSD Q?
+L Device:Q_NMOS_GDSD Q2
 U 1 1 60967E49
 P 4425 1850
-F 0 "Q?" V 4325 1775 50  0000 C CNN
+F 0 "Q2" V 4325 1775 50  0000 C CNN
 F 1 "NTD5865NL" V 4225 1625 50  0000 C CNN
 F 2 "Package_TO_SOT_SMD:TO-252-3_TabPin4" H 4625 1950 50  0001 C CNN
@@
 	7650 2325 7650 2250
 $Comp
-L Device:R_Small_US R?
+L Device:R_Small_US R41
 U 1 1 60ADCC0E
 P 10575 1850
-F 0 "R?" H 10650 1875 50  0000 L CNN
+F 0 "R41" H 10650 1875 50  0000 L CNN
 F 1 "100K" H 10625 1800 50  0000 L CNN
-F 2 "" H 10575 1850 50  0001 C CNN
+F 2 "Resistor_SMD:R_0805_2012Metric_Pad1.20x1.40mm_HandSolder" H 10575 1850 50  0001 C CNN
 F 3 "~" H 10575 1850 50  0001 C CNN
 	1    10575 1850
@@
 $EndComp
 $Comp
-L Device:R_Small_US R?
+L Device:R_Small_US R43
 U 1 1 60ADCFBE
 P 10200 2000
-F 0 "R?" V 10350 1950 50  0000 L CNN
+F 0 "R43" V 10350 1950 50  0000 L CNN
 F 1 "100R" V 10275 1900 50  0000 L CNN
-F 2 "" H 10200 2000 50  0001 C CNN
+F 2 "Resistor_SMD:R_0805_2012Metric_Pad1.20x1.40mm_HandSolder" H 10200 2000 50  0001 C CNN
 F 3 "~" H 10200 2000 50  0001 C CNN
 	1    10200 2000
@@
 $EndComp
 $Comp
-L Device:R_Small_US R?
+L Device:R_Small_US R44
 U 1 1 60ADD5C0
 P 10350 2100
-F 0 "R?" H 10150 2025 50  0000 L CNN
+F 0 "R44" H 10150 2025 50  0000 L CNN
 F 1 "100K" H 10125 1950 50  0000 L CNN
-F 2 "" H 10350 2100 50  0001 C CNN
+F 2 "Resistor_SMD:R_0805_2012Metric_Pad1.20x1.40mm_HandSolder" H 10350 2100 50  0001 C CNN
 F 3 "~" H 10350 2100 50  0001 C CNN
 	1    10350 2100
@@
 $EndComp
 $Comp
-L MAGI_Symbols:LTC2966CSWPBF U?
+L MAGI_Symbols:LTC2966CSWPBF U13
 U 1 1 606D1CF4
 P 7650 1650
-F 0 "U?" H 9200 2025 50  0000 C CNN
+F 0 "U13" H 9200 2025 50  0000 C CNN
 F 1 "LTC2966CSWPBF" H 9475 1925 50  0000 C CNN
 F 2 "MAGI_Footprints:SO-20_SW" H 9750 1800 50  0001 L BNN
@@
 $EndComp
 $Comp
-L Device:R_Small_US R?
+L Device:R_Small_US R39
 U 1 1 60ACAE5C
 P 10300 1700
-F 0 "R?" V 10150 1700 50  0000 C CNN
+F 0 "R39" V 10150 1700 50  0000 C CNN
 F 1 "100R" V 10225 1700 50  0000 C CNN
-F 2 "" H 10300 1700 50  0001 C CNN
+F 2 "Resistor_SMD:R_0805_2012Metric_Pad1.20x1.40mm_HandSolder" H 10300 1700 50  0001 C CNN
 F 3 "~" H 10300 1700 50  0001 C CNN
 	1    10300 1700
@@
 $EndComp
 $Comp
-L power:GND #PWR?
+L power:GND #PWR082
 U 1 1 60B7B134
 P 10350 2275
-F 0 "#PWR?" H 10350 2025 50  0001 C CNN
+F 0 "#PWR082" H 10350 2025 50  0001 C CNN
 F 1 "GND" H 10355 2102 50  0000 C CNN
 F 2 "" H 10350 2275 50  0001 C CNN
@@
 	10350 2275 10350 2200
 $Comp
-L power:GND #PWR?
+L power:GND #PWR083
 U 1 1 60BBBFAA
 P 10575 2275
-F 0 "#PWR?" H 10575 2025 50  0001 C CNN
+F 0 "#PWR083" H 10575 2025 50  0001 C CNN
 F 1 "GND" H 10580 2102 50  0000 C CNN
 F 2 "" H 10575 2275 50  0001 C CNN
