File: SMU Test Fixture/power_supplies.sch (KiCad schematic (older format))
At the start: 54 parts, among them J13 Hot_Spade, J14 Power Outputs, J15 Neutral_Spade, Q1 NTD5865NL, Q2 NTD5865NL, T1 VPP28-1060, U10 LT3045, U11 LT1086-12, U12 LT3094, U13 LTC2966CSWPBF, U9 LT1086-5.0

Commit message: Switch to QFN package for LTC2966.
Parts:
- R39, R40, R41, R42, R43, R44, R45, R46, R47, R48: footprint Resistor_SMD:R_0805_2012Metric_Pad1.20x1.40mm_HandSolder -> Resistor_SMD:R_0603_1608Metric_Pad0.98x0.95mm_HandSolder
- U13: footprint MAGI_Footprints:SO-20_SW -> Package_DFN_QFN:QFN-16-1EP_3x3mm_P0.5mm_EP1.45x1.45mm; symbol MAGI_Symbols:LTC2966CSWPBF -> MAGI_Symbols:LTC2966_QFN
Connections:
- wire segments 256 -> 258
Changed lines of the file:
@@
 F 0 "R45" H 7368 2246 50  0000 L CNN
 F 1 "4.02k" H 7368 2155 50  0000 L CNN
-F 2 "Resistor_SMD:R_0805_2012Metric_Pad1.20x1.40mm_HandSolder" H 7300 2200 50  0001 C CNN
+F 2 "Resistor_SMD:R_0603_1608Metric_Pad0.98x0.95mm_HandSolder" H 7300 2200 50  0001 C CNN
 F 3 "~" H 7300 2200 50  0001 C CNN
 	1    7300 2200
@@
 F 0 "R47" H 7368 2496 50  0000 L CNN
 F 1 "845R" H 7368 2405 50  0000 L CNN
-F 2 "Resistor_SMD:R_0805_2012Metric_Pad1.20x1.40mm_HandSolder" H 7300 2450 50  0001 C CNN
+F 2 "Resistor_SMD:R_0603_1608Metric_Pad0.98x0.95mm_HandSolder" H 7300 2450 50  0001 C CNN
 F 3 "~" H 7300 2450 50  0001 C CNN
 	1    7300 2450
@@
 F 0 "R48" H 7368 2746 50  0000 L CNN
 F 1 "46.4K" H 7368 2655 50  0000 L CNN
-F 2 "Resistor_SMD:R_0805_2012Metric_Pad1.20x1.40mm_HandSolder" H 7300 2700 50  0001 C CNN
+F 2 "Resistor_SMD:R_0603_1608Metric_Pad0.98x0.95mm_HandSolder" H 7300 2700 50  0001 C CNN
 F 3 "~" H 7300 2700 50  0001 C CNN
 	1    7300 2700
@@
 F 0 "R40" H 6918 1796 50  0000 L CNN
 F 1 "4.96K" H 6918 1705 50  0000 L CNN
-F 2 "Resistor_SMD:R_0805_2012Metric_Pad1.20x1.40mm_HandSolder" H 6850 1750 50  0001 C CNN
+F 2 "Resistor_SMD:R_0603_1608Metric_Pad0.98x0.95mm_HandSolder" H 6850 1750 50  0001 C CNN
 F 3 "~" H 6850 1750 50  0001 C CNN
 	1    6850 1750
@@
 F 0 "R42" H 6918 2046 50  0000 L CNN
 F 1 "46.4K" H 6918 1955 50  0000 L CNN
-F 2 "Resistor_SMD:R_0805_2012Metric_Pad1.20x1.40mm_HandSolder" H 6850 2000 50  0001 C CNN
+F 2 "Resistor_SMD:R_0603_1608Metric_Pad0.98x0.95mm_HandSolder" H 6850 2000 50  0001 C CNN
 F 3 "~" H 6850 2000 50  0001 C CNN
 	1    6850 2000
@@
 F 0 "R46" H 6918 2296 50  0000 L CNN
 F 1 "4.64K" H 6918 2205 50  0000 L CNN
-F 2 "Resistor_SMD:R_0805_2012Metric_Pad1.20x1.40mm_HandSolder" H 6850 2250 50  0001 C CNN
+F 2 "Resistor_SMD:R_0603_1608Metric_Pad0.98x0.95mm_HandSolder" H 6850 2250 50  0001 C CNN
 F 3 "~" H 6850 2250 50  0001 C CNN
 	1    6850 2250
@@
 F 0 "R41" H 10650 1875 50  0000 L CNN
 F 1 "100K" H 10625 1800 50  0000 L CNN
-F 2 "Resistor_SMD:R_0805_2012Metric_Pad1.20x1.40mm_HandSolder" H 10575 1850 50  0001 C CNN
+F 2 "Resistor_SMD:R_0603_1608Metric_Pad0.98x0.95mm_HandSolder" H 10575 1850 50  0001 C CNN
 F 3 "~" H 10575 1850 50  0001 C CNN
 	1    10575 1850
@@
 F 0 "R43" V 10350 1950 50  0000 L CNN
 F 1 "100R" V 10275 1900 50  0000 L CNN
-F 2 "Resistor_SMD:R_0805_2012Metric_Pad1.20x1.40mm_HandSolder" H 10200 2000 50  0001 C CNN
+F 2 "Resistor_SMD:R_0603_1608Metric_Pad0.98x0.95mm_HandSolder" H 10200 2000 50  0001 C CNN
 F 3 "~" H 10200 2000 50  0001 C CNN
 	1    10200 2000
@@
 F 0 "R44" H 10150 2025 50  0000 L CNN
 F 1 "100K" H 10125 1950 50  0000 L CNN
-F 2 "Resistor_SMD:R_0805_2012Metric_Pad1.20x1.40mm_HandSolder" H 10350 2100 50  0001 C CNN
+F 2 "Resistor_SMD:R_0603_1608Metric_Pad0.98x0.95mm_HandSolder" H 10350 2100 50  0001 C CNN
 F 3 "~" H 10350 2100 50  0001 C CNN
 	1    10350 2100
@@
 $EndComp
 $Comp
-L MAGI_Symbols:LTC2966CSWPBF U13
+L MAGI_Symbols:LTC2966_QFN U13
 U 1 1 606D1CF4
 P 7650 1650
 F 0 "U13" H 9200 2025 50  0000 C CNN
 F 1 "LTC2966CSWPBF" H 9475 1925 50  0000 C CNN
-F 2 "MAGI_Footprints:SO-20_SW" H 9750 1800 50  0001 L BNN
+F 2 "Package_DFN_QFN:QFN-16-1EP_3x3mm_P0.5mm_EP1.45x1.45mm" H 9750 1800 50  0001 L BNN
 F 3 "" H 9750 1300 50  0001 L BNN
 F 4 "Linear Technology" H 9650 2000 50  0001 L BNN "VENDOR"
@@
 F 0 "R39" V 10150 1700 50  0000 C CNN
 F 1 "100R" V 10225 1700 50  0000 C CNN
-F 2 "Resistor_SMD:R_0805_2012Metric_Pad1.20x1.40mm_HandSolder" H 10300 1700 50  0001 C CNN
+F 2 "Resistor_SMD:R_0603_1608Metric_Pad0.98x0.95mm_HandSolder" H 10300 1700 50  0001 C CNN
 F 3 "~" H 10300 1700 50  0001 C CNN
 	1    10300 1700
@@
 	10575 1700 10725 1700
 Connection ~ 3650 2300
+Wire Wire Line
+	10050 2450 10050 3100
+Wire Wire Line
+	10050 3100 9725 3100
+Connection ~ 9725 3100
 $EndSCHEMATC
