File: SMU Test Fixture/shunts.sch (KiCad schematic (older format))
At the start: 9 parts

Commit message: Add analog switch power connections.
Parts:
- added C? (x4): 100n, Capacitor_SMD:C_0805_2012Metric_Pad1.18x1.45mm_HandSolder, symbol Device:C_Small
- added C? (x2): 1u, symbol Device:C_Small
- added R? (x2): 100R, symbol Device:R_Small_US
Connections:
- net labels added: +15V, -15V, GND
- wire segments 78 -> 112
