File: SMU Test Fixture/SMUTestFixture.sch (KiCad schematic (older format))
At the start: 34 parts

Commit message: Add analog switch power connections.
Parts:
- removed R?: 56K, Resistor_SMD:R_0805_2012Metric_Pad1.20x1.40mm_HandSolder, symbol Device:R_Small_US
- added C?: 1u, symbol Device:C_Small
- added D?: Vcl=14V, Diode_SMD:D_0201_0603Metric_Pad0.64x0.40mm_HandSolder, symbol Device:D_TVS
- added R? (x3): 100R, symbol Device:R_Small_US
Connections:
- net labels added: wg_1
- net labels removed: IV_src_input
- wire segments 135 -> 158
Other:
- moved on the sheet: C?, Q?

Commit message: Add new shunt amp design to SMU schematic.
Parts:
- removed R?: 1M, symbol Device:R_Small_US
- removed R?: 20K, symbol Device:R_Small_US
- removed U?: THS4021CxDGNx, Package_SO:TI_SO-PowerPAD-8, symbol MAGI_Symbols:THS4021CxDGNx
- added C?: 1u, symbol Device:C_Small
- added R?: 430R, Resistor_SMD:R_0805_2012Metric_Pad1.20x1.40mm_HandSolder, symbol Device:R_Small_US
- added R? (x2): 4.3K, symbol Device:R_Small_US
- added R?: 430R, symbol Device:R_Small_US
- added U? (x3): THS3092D, Package_SO:SOIC-8_3.9x4.9mm_P1.27mm, symbol MAGI_Symbols:THS3092D
- R? (x2): value 1.47K -> 14.7K
- R?: value 15R -> 150R
Connections:
- wire segments 158 -> 170
- no-connect marks 3 -> 1
Other:
- moved on the sheet: R?
