File: SMU Test Fixture/SMUTestFixture.kicad_sch (KiCad schematic)
At the start: 49 parts, among them K1 EE2-12SNU, Q1 BCP56, Q2 BCP56, U1 THS3092D, U2 OPA189IDBVx, U3 OPA189IDBVx, U4 ADGS1412, U5 OPA192IDBVx, U6 OPA192IDBVx, U7 OPA189IDBVx, U8 OPA551U, U9 ADGS1412

Commit message: Initial commit
Other:
- note added: ".010"/0.050" grid"
- note removed: ".010" grid"
Changed lines of the file:
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@@
     (stroke (width 0) (type default) (color 0 0 0 0))
   )
-  (text ".010\" grid" (at 178.562 169.418 0)
+  (text ".010\"/0.050\" grid" (at 178.562 169.418 0)
     (effects (font (size 1.27 1.27)) (justify left bottom))
   )
-  (text "Current Shunt Amplifier" (at 35.56 167.64 0)
+  (text "Current Shunt Amplifier" (at 14.478 102.362 0)
     (effects (font (size 1.4986 1.4986) (thickness 0.2997) bold) (justify left bottom))
   )
