File: SMU Shunt Amp/SMU Shunt Amp.sch (KiCad schematic (older format))
At the start: 30 parts, among them J1 30VDC, J2 Input, J3 Output, U1 OPA189IDBVx, U2 THS3092D

Commit message: Add ferrites
Parts:
- added FB1, FB2: 80R @ 100MHz, Resistor_SMD:R_1206_3216Metric_Pad1.30x1.75mm_HandSolder, symbol Device:Ferrite_Bead_Small
- C8: value Optional -> 1u
Connections:
- net +15V: now also FB1.2; no longer D1.1 (K), D3.1 (K)
- net -15V: now also FB2.2; no longer D2.2 (A), D3.2 (A)
- new net: D2.2 (A), D3.2 (A), FB2.1
- new net: D1.1 (K), D3.1 (K), FB1.1
Other:
- moved on the sheet: C5, C6
Changed lines of the file:
@@
 L MAGI_Symbols:-14V #PWR08
 U 1 1 60586099
-P 2925 2200
-F 0 "#PWR08" H 2925 2300 50  0001 C CNN
-F 1 "-14V" H 2940 2373 50  0000 C CNN
-F 2 "" H 2925 2200 50  0001 C CNN
-F 3 "" H 2925 2200 50  0001 C CNN
-	1    2925 2200
+P 3300 2200
+F 0 "#PWR08" H 3300 2300 50  0001 C CNN
+F 1 "-14V" H 3315 2373 50  0000 C CNN
+F 2 "" H 3300 2200 50  0001 C CNN
+F 3 "" H 3300 2200 50  0001 C CNN
+	1    3300 2200
 	-1   0    0    1
 $EndComp
@@
 L MAGI_Symbols:+14V #PWR07
 U 1 1 60583414
-P 2925 1425
-F 0 "#PWR07" H 2925 1275 50  0001 C CNN
-F 1 "+14V" H 2940 1598 50  0000 C CNN
-F 2 "" H 2925 1425 50  0001 C CNN
-F 3 "" H 2925 1425 50  0001 C CNN
-	1    2925 1425
+P 3300 1425
+F 0 "#PWR07" H 3300 1275 50  0001 C CNN
+F 1 "+14V" H 3315 1598 50  0000 C CNN
+F 2 "" H 3300 1425 50  0001 C CNN
+F 3 "" H 3300 1425 50  0001 C CNN
+	1    3300 1425
 	1    0    0    -1
 $EndComp
@@
 L Device:CP1_Small C6
 U 1 1 607C786C
-P 2925 1975
-F 0 "C6" H 3016 2021 50  0000 L CNN
-F 1 "10u" H 3016 1930 50  0000 L CNN
-F 2 "Capacitor_SMD:CP_Elec_6.3x7.7" H 2925 1975 50  0001 C CNN
-F 3 "https://www.mouser.com/datasheet/2/293/e_ucz-1903374.pdf" H 2925 1975 50  0001 C CNN
-F 4 "UCZ1J100MCS1GS" H 2925 1975 50  0001 C CNN "Part"
-	1    2925 1975
+P 3300 1975
+F 0 "C6" H 3391 2021 50  0000 L CNN
+F 1 "10u" H 3391 1930 50  0000 L CNN
+F 2 "Capacitor_SMD:CP_Elec_6.3x7.7" H 3300 1975 50  0001 C CNN
+F 3 "https://www.mouser.com/datasheet/2/293/e_ucz-1903374.pdf" H 3300 1975 50  0001 C CNN
+F 4 "UCZ1J100MCS1GS" H 3300 1975 50  0001 C CNN "Part"
+	1    3300 1975
 	1    0    0    -1
 $EndComp
@@
 L Device:CP1_Small C5
 U 1 1 607C2943
-P 2925 1650
-F 0 "C5" H 3016 1696 50  0000 L CNN
-F 1 "10u" H 3016 1605 50  0000 L CNN
-F 2 "Capacitor_SMD:CP_Elec_6.3x7.7" H 2925 1650 50  0001 C CNN
-F 3 "https://www.mouser.com/datasheet/2/293/e_ucz-1903374.pdf" H 2925 1650 50  0001 C CNN
-F 4 "UCZ1J100MCS1GS" H 2925 1650 50  0001 C CNN "Part"
-	1    2925 1650
-	1    0    0    -1
-$EndComp
-Wire Wire Line
-	2925 1800 2925 1875
-Wire Wire Line
-	3575 1800 3575 1825
-Wire Wire Line
-	2925 1800 3575 1800
-Wire Wire Line
-	2925 2075 2925 2200
-Connection ~ 2925 1800
-Wire Wire Line
-	2925 1750 2925 1800
-Wire Wire Line
-	2925 1425 2925 1550
+P 3300 1650
+F 0 "C5" H 3391 1696 50  0000 L CNN
+F 1 "10u" H 3391 1605 50  0000 L CNN
+F 2 "Capacitor_SMD:CP_Elec_6.3x7.7" H 3300 1650 50  0001 C CNN
+F 3 "https://www.mouser.com/datasheet/2/293/e_ucz-1903374.pdf" H 3300 1650 50  0001 C CNN
+F 4 "UCZ1J100MCS1GS" H 3300 1650 50  0001 C CNN "Part"
+	1    3300 1650
+	1    0    0    -1
+$EndComp
+Wire Wire Line
+	3300 1800 3300 1875
+Wire Wire Line
+	3950 1800 3950 1825
+Wire Wire Line
+	3300 1800 3950 1800
+Wire Wire Line
+	3300 2075 3300 2200
+Connection ~ 3300 1800
+Wire Wire Line
+	3300 1750 3300 1800
+Wire Wire Line
+	3300 1425 3300 1550
 $Comp
 L power:GND #PWR010
 U 1 1 60594A7B
-P 3575 1825
-F 0 "#PWR010" H 3575 1575 50  0001 C CNN
-F 1 "GND" H 3580 1652 50  0000 C CNN
-F 2 "" H 3575 1825 50  0001 C CNN
-F 3 "" H 3575 1825 50  0001 C CNN
-	1    3575 1825
+P 3950 1825
+F 0 "#PWR010" H 3950 1575 50  0001 C CNN
+F 1 "GND" H 3955 1652 50  0000 C CNN
+F 2 "" H 3950 1825 50  0001 C CNN
+F 3 "" H 3950 1825 50  0001 C CNN
+	1    3950 1825
 	1    0    0    -1
 $EndComp
@@
 L MAGI_Symbols:+14V #PWR05
 U 1 1 60991141
-P 2425 1575
-F 0 "#PWR05" H 2425 1425 50  0001 C CNN
-F 1 "+14V" H 2440 1748 50  0000 C CNN
-F 2 "" H 2425 1575 50  0001 C CNN
-F 3 "" H 2425 1575 50  0001 C CNN
-	1    2425 1575
+P 2875 1575
+F 0 "#PWR05" H 2875 1425 50  0001 C CNN
+F 1 "+14V" H 2890 1748 50  0000 C CNN
+F 2 "" H 2875 1575 50  0001 C CNN
+F 3 "" H 2875 1575 50  0001 C CNN
+	1    2875 1575
 	1    0    0    -1
 $EndComp
@@
 L MAGI_Symbols:-14V #PWR06
 U 1 1 60991147
-P 2425 2000
-F 0 "#PWR06" H 2425 2100 50  0001 C CNN
-F 1 "-14V" H 2440 2173 50  0000 C CNN
-F 2 "" H 2425 2000 50  0001 C CNN
-F 3 "" H 2425 2000 50  0001 C CNN
-	1    2425 2000
+P 2875 2000
+F 0 "#PWR06" H 2875 2100 50  0001 C CNN
+F 1 "-14V" H 2890 2173 50  0000 C CNN
+F 2 "" H 2875 2000 50  0001 C CNN
+F 3 "" H 2875 2000 50  0001 C CNN
+	1    2875 2000
 	-1   0    0    1
 $EndComp
@@
 P 4400 2825
 F 0 "C8" V 4171 2825 50  0000 C CNN
-F 1 "Optional" V 4262 2825 50  0000 C CNN
+F 1 "1u" V 4262 2825 50  0000 C CNN
 F 2 "Capacitor_SMD:C_0805_2012Metric_Pad1.18x1.45mm_HandSolder" H 4400 2825 50  0001 C CNN
 F 3 "~" H 4400 2825 50  0001 C CNN
@@
 U 1 1 60AE7844
 P 2250 1800
-F 0 "D3" V 2204 1870 50  0000 L CNN
+F 0 "D3" V 2175 1850 50  0000 L CNN
 F 1 "Vz=30" V 2295 1870 50  0000 L CNN
 F 2 "Diode_SMD:D_SOD-123" V 2250 1800 50  0001 C CNN
@@
 Wire Wire Line
 	2250 1700 2250 1575
+Wire Wire Line
+	2250 1900 2250 2000
+Wire Wire Line
+	5550 3325 5775 3325
+$Comp
+L Device:Ferrite_Bead_Small FB1
+U 1 1 60D3E83B
+P 2450 1575
+F 0 "FB1" V 2687 1575 50  0000 C CNN
+F 1 "80R @ 100MHz" V 2596 1575 50  0000 C CNN
+F 2 "Resistor_SMD:R_1206_3216Metric_Pad1.30x1.75mm_HandSolder" V 2380 1575 50  0001 C CNN
+F 3 "https://www.mouser.com/datasheet/2/987/Laird_10092020_Laird_MCP_Catalog_EMI_Filtering_and-1947796.pdf" H 2450 1575 50  0001 C CNN
+F 4 "HI1206N800R-10" H 2450 1575 50  0001 C CNN "PN"
+	1    2450 1575
+	0    -1   -1   0
+$EndComp
+Wire Wire Line
+	2350 2000 2250 2000
+Connection ~ 2250 2000
+Wire Wire Line
+	2550 2000 2875 2000
+Wire Wire Line
+	2250 1575 2350 1575
 Connection ~ 2250 1575
 Wire Wire Line
-	2250 1575 2425 1575
-Wire Wire Line
-	2250 1900 2250 2000
-Connection ~ 2250 2000
-Wire Wire Line
-	2250 2000 2425 2000
-Wire Wire Line
-	5550 3325 5775 3325
+	2550 1575 2875 1575
+$Comp
+L Device:Ferrite_Bead_Small FB2
+U 1 1 60D60535
+P 2450 2000
+F 0 "FB2" V 2300 2025 50  0000 C CNN
+F 1 "80R @ 100MHz" V 2225 2000 50  0000 C CNN
+F 2 "Resistor_SMD:R_1206_3216Metric_Pad1.30x1.75mm_HandSolder" V 2380 2000 50  0001 C CNN
+F 3 "https://www.mouser.com/datasheet/2/987/Laird_10092020_Laird_MCP_Catalog_EMI_Filtering_and-1947796.pdf" H 2450 2000 50  0001 C CNN
+F 4 "HI1206N800R-10" H 2450 2000 50  0001 C CNN "PN"
+	1    2450 2000
+	0    -1   -1   0
+$EndComp
 $EndSCHEMATC
